File: LED Controller.kicad_pcb (KiCad board)
At the start: 2 copper layers, 59.7 x 58.3 mm, 22 parts, among them J1 Conn_01x03, J2 Conn_01x03, J3 Conn_01x03, J4 Conn_01x03, J5 Conn_01x03, J6 12v IN, J7 SPI, J8 Conn_01x02, U1 4504, U2 L7805

Commit message: Add export
Parts:
- added C2: 0.33u, Capacitor_THT:CP_Radial_D4.0mm_P1.50mm, F.Cu at (167.5, 96.8)
- moved J7 0.92 mm to (172.1, 92.2)
Routing:
- net /12V: track 90.5 -> 92.0 mm
- net /SPI1_MOSI: track 40.8 -> 41.6 mm
- net /SPI1_MISO: track 40.5 -> 41.1 mm
- net /SPI1_NSS: track 50.4 -> 50.9 mm
